File: hardware/3_phase_inverter_board/3_ph_inv_brd--pwr.sch (KiCad schematic (older format))
At the start: 10 parts

Commit message: Edited a little more than placed order!
Parts:
- added C18, C22: 100nF, symbol Device:C_Small
- added C19, C20, C23: 10uF, symbol Device:C_Small
- added C24, C25, C26: 56uF, symbol Device:CP
- added C29: 15nF, symbol Device:C_Small
- added C30: 820pF, symbol Device:C_Small
- added C31: 10pF, symbol Device:C_Small
- added D2: 10A 960mV, symbol Device:D_Schottky
- added J2: XT60, symbol Connector:Conn_01x02_Female
- added L2: 6.8uH 8.1mOhm, symbol Device:L
- added Q8: CSD18534KCS, symbol 3_phase_inverter_board:CSD18534KCS
- added R16: 1k, symbol Device:R_Small
- added R17, R19: 10k, symbol Device:R_Small
- added R18, R23: 30.9k, symbol Device:R_Small
- added R20: 100, symbol Device:R_Small
- added R21: 5mOhms, symbol Device:R_Small
- added R22: 6.19k, symbol Device:R_Small
- added U10: LM3478, symbol 3_phase_inverter_board:LM3478
- added U6: L7812, symbol Regulator_Linear:L7812
- added U8: LD1117AVCC, symbol 3_phase_inverter_board:LD1117AVCC
- added U9: MCP602, symbol Amplifier_Operational:MCP602
- gave numbers to parts that had none: 10
Connections:
- net GND: now also C27.2, C28.2, C18.2, C19.2, C20.2, C22.2, C23.2, C24.2, C25.2, C26.2, C30.2, C31.2, J2.2 (Pin_2), R16.1, R19.1, R21.2, R22.2, R23.2, U10.4 (AGND), U10.5 (PGND), U6.2 (GND), U8.1 (GND), U9.4 (V-), U9.6 (-)
- net INPUT_S+: now also C20.1
- net INPUT_S-: now also C27.1, C28.1, L2.1, U10.8 (VIN)
- new net: C31.1, R20.2, U10.1 (ISENSE)
- new net: C29.1, C30.1, U10.2 (COMP)
- new net: R16.2, R18.2, U10.3 (FB)
- new net: Q8.1 (G), U10.6 (DR)
- new net: R23.1, U10.~ (FA/SD)
- new net: C29.2, R22.1
- new net: D2.2 (A), L2.2, Q8.2 (D)
- new net: Q8.3 (S), R20.1, R21.1
- new net: R17.1, R19.2, U9.3 (+)
- new net +12V: C19.1, C22.1, U6.3 (OUT), U8.3 (VI)
- new net +3V3: C23.1, R17.2, U8.2 (VO), U9.5 (+), U9.8 (V+)
- new net 1.65VREF: U9.1, U9.2 (-)
- new net VBUS: C24.1, C25.1, C26.1, D2.1 (K), R18.1
- new net VS: C18.1, J2.1 (Pin_1), U6.1 (IN)
- no-connect marks 1 -> 2
Other:
- note added: "3V3 AND +12V POWER"
- note added: "BOOST CONVERTER STAGE: VBAT --> 40VDC"
- note added: "R_FA = 4.503e11 x Fpwm^-1.26\nChosen frequency : 485 kHz"
- note added: "VBAT INPUT"
- note added: "Virtual 1.65V Node"
- note removed: "VBAT"
- moved on the sheet: C27, C28
