File: hardware/3_phase_inverter_board/3_phase_inverter_board.sch (KiCad schematic (older format))
At the start: 45 parts, among them J101 Conn_01x05_Male, Y101 10MHz

Commit message: Edited a little more than placed order!
Parts:
- gave numbers to parts that had none: 30
- renumbered C101 to C1, C104 to C10, C106 to C11, C107 to C12, C105 to C14, C108 to C15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
